File: Costume Controller Base Board.sch (EAGLE design)
At the start: 38 parts, among them J1 USB MICRO, U1 ATMEGA32U4-XUMU, U2 PCA9306DCUT, U3 LP2985-33DBVR, U4 MPU-6050-1, U5 TPS61200, X1 09FLZ-SM1, Y1 16MHz KX-7

Commit message: added pullups
Parts:
- removed X1: 09FLZ-SM1, con-jst:09FLZ-SM1
- added R11, R12: 10k, SparkFun:RESISTOR0603-RES
Connections:
- new net SCL1: R4.1, R5.1
- net N$2: now also R11.2, R12.2
- net SCL2: now also R11.1
- net SDA2: now also R12.1
- net STRAND1: no longer X1-1.1
- net STRAND4: no longer X1-4.1
- net STRAND5: no longer X1-5.1
- net STRAND6: no longer X1-6.1
- net STRAND7: no longer X1-7.1
- net STRAND9: no longer X1-9.1
Other:
- note removed: "JST Connector 9 pin"
Changed lines of the file:
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@@
 <part name="GND9" library="SparkFun" deviceset="GND" device=""/>
 <part name="GND10" library="SparkFun" deviceset="GND" device=""/>
-<part name="X1" library="con-jst" deviceset="09FLZ-SM1" device=""/>
+<part name="R11" library="SparkFun" deviceset="RESISTOR" device="0603-RES" value="10k"/>
+<part name="R12" library="SparkFun" deviceset="RESISTOR" device="0603-RES" value="10k"/>
 </parts>
 <sheets>
@@
 <text x="-1013.46" y="261.62" size="1.778" layer="97">ENABLE tied high, could be IO</text>
 <text x="-1013.46" y="261.62" size="1.778" layer="97">ENABLE tied high, could be IO</text>
-<text x="-797.56" y="180.34" size="1.778" layer="97">JST Connector 9 pin</text>
 </plain>
 <instances>
@@
 <instance part="GND9" gate="1" x="-1033.78" y="259.08"/>
 <instance part="GND10" gate="1" x="-1054.1" y="228.6"/>
-<instance part="X1" gate="-1" x="-769.62" y="170.18"/>
-<instance part="X1" gate="-2" x="-769.62" y="167.64"/>
-<instance part="X1" gate="-3" x="-769.62" y="165.1"/>
-<instance part="X1" gate="-4" x="-769.62" y="162.56"/>
-<instance part="X1" gate="-5" x="-769.62" y="160.02"/>
-<instance part="X1" gate="-6" x="-769.62" y="157.48"/>
-<instance part="X1" gate="-7" x="-769.62" y="154.94"/>
-<instance part="X1" gate="-8" x="-769.62" y="152.4"/>
-<instance part="X1" gate="-9" x="-769.62" y="149.86"/>
+<instance part="R11" gate="G$1" x="-952.5" y="248.92" rot="R90"/>
+<instance part="R12" gate="G$1" x="-942.34" y="248.92" rot="R90"/>
 </instances>
 <busses>
@@
 <pinref part="U1" gate="G$1" pin="(OC0B/SCL/INT0)PD0"/>
 <wire x1="-741.68" y1="251.46" x2="-741.68" y2="213.36" width="0.1524" layer="91"/>
-<wire x1="-741.68" y1="213.36" x2="-980.44" y2="213.36" width="0.1524" layer="91"/>
+<wire x1="-741.68" y1="213.36" x2="-952.5" y2="213.36" width="0.1524" layer="91"/>
+<wire x1="-952.5" y1="213.36" x2="-980.44" y2="213.36" width="0.1524" layer="91"/>
 <wire x1="-980.44" y1="213.36" x2="-980.44" y2="238.76" width="0.1524" layer="91"/>
 <wire x1="-980.44" y1="238.76" x2="-1005.84" y2="238.76" width="0.1524" layer="91"/>
+<pinref part="R11" gate="G$1" pin="1"/>
+<wire x1="-952.5" y1="243.84" x2="-952.5" y2="213.36" width="0.1524" layer="91"/>
+<junction x="-952.5" y="213.36"/>
 </segment>
 </net>
@@
 <pinref part="U1" gate="G$1" pin="(SDA/INT1)PD1"/>
 <wire x1="-734.06" y1="254" x2="-734.06" y2="210.82" width="0.1524" layer="91"/>
-<wire x1="-734.06" y1="210.82" x2="-982.98" y2="210.82" width="0.1524" layer="91"/>
+<wire x1="-734.06" y1="210.82" x2="-942.34" y2="210.82" width="0.1524" layer="91"/>
+<wire x1="-942.34" y1="210.82" x2="-982.98" y2="210.82" width="0.1524" layer="91"/>
 <wire x1="-982.98" y1="210.82" x2="-982.98" y2="236.22" width="0.1524" layer="91"/>
 <wire x1="-982.98" y1="236.22" x2="-1005.84" y2="236.22" width="0.1524" layer="91"/>
+<pinref part="R12" gate="G$1" pin="1"/>
+<wire x1="-942.34" y1="243.84" x2="-942.34" y2="210.82" width="0.1524" layer="91"/>
+<junction x="-942.34" y="210.82"/>
 </segment>
 </net>
@@
 <net name="SCL1" class="0">
 <segment>
-<wire x1="-1127.76" y1="220.98" x2="-993.14" y2="220.98" width="0.1524" layer="91"/>
+<wire x1="-1127.76" y1="220.98" x2="-1104.9" y2="220.98" width="0.1524" layer="91"/>
+<wire x1="-1104.9" y1="220.98" x2="-1097.28" y2="220.98" width="0.1524" layer="91"/>
+<wire x1="-1097.28" y1="220.98" x2="-993.14" y2="220.98" width="0.1524" layer="91"/>
 <wire x1="-993.14" y1="220.98" x2="-993.14" y2="246.38" width="0.1524" layer="91"/>
 <wire x1="-993.14" y1="246.38" x2="-1005.84" y2="246.38" width="0.1524" layer="91"/>
+<pinref part="R5" gate="G$1" pin="1"/>
+<wire x1="-1097.28" y1="231.14" x2="-1097.28" y2="220.98" width="0.1524" layer="91"/>
+<pinref part="R4" gate="G$1" pin="1"/>
+<wire x1="-1104.9" y1="231.14" x2="-1104.9" y2="220.98" width="0.1524" layer="91"/>
+<junction x="-1104.9" y="220.98"/>
+<junction x="-1097.28" y="220.98"/>
 </segment>
 </net>
@@
 <junction x="-1054.1" y="243.84"/>
 <junction x="-1033.78" y="281.94"/>
+<wire x1="-1033.78" y1="281.94" x2="-952.5" y2="281.94" width="0.1524" layer="91"/>
+<wire x1="-952.5" y1="281.94" x2="-942.34" y2="281.94" width="0.1524" layer="91"/>
+<wire x1="-952.5" y1="281.94" x2="-952.5" y2="254" width="0.1524" layer="91"/>
+<wire x1="-942.34" y1="281.94" x2="-942.34" y2="254" width="0.1524" layer="91"/>
+<pinref part="R11" gate="G$1" pin="2"/>
+<pinref part="R12" gate="G$1" pin="2"/>
 </segment>
 </net>
@@
 <label x="-741.68" y="256.54" size="1.27" layer="95" xref="yes"/>
 </segment>
-<segment>
-<pinref part="X1" gate="-1" pin="1"/>
-<wire x1="-774.7" y1="170.18" x2="-792.48" y2="170.18" width="0.1524" layer="91"/>
-<label x="-792.48" y="170.18" size="1.27" layer="95" rot="MR0" xref="yes"/>
-</segment>
 </net>
 <net name="STRAND2" class="0">
@@
 <label x="-741.68" y="259.08" size="1.27" layer="95" xref="yes"/>
 </segment>
-<segment>
-<wire x1="-772.16" y1="167.64" x2="-792.48" y2="167.64" width="0.1524" layer="91"/>
-<label x="-792.48" y="167.64" size="1.27" layer="95" rot="MR0" xref="yes"/>
-</segment>
 </net>
 <net name="STRAND3" class="0">
@@
 <label x="-741.68" y="261.62" size="1.27" layer="95" xref="yes"/>
 </segment>
-<segment>
-<wire x1="-772.16" y1="165.1" x2="-792.48" y2="165.1" width="0.1524" layer="91"/>
-<label x="-792.48" y="165.1" size="1.27" layer="95" rot="MR0" xref="yes"/>
-</segment>
 </net>
 <net name="STRAND4" class="0">
@@
 <label x="-741.68" y="264.16" size="1.27" layer="95" xref="yes"/>
 </segment>
-<segment>
-<pinref part="X1" gate="-4" pin="1"/>
-<wire x1="-774.7" y1="162.56" x2="-792.48" y2="162.56" width="0.1524" layer="91"/>
-<label x="-792.48" y="162.56" size="1.27" layer="95" rot="MR0" xref="yes"/>
-</segment>
 </net>
 <net name="STRAND5" class="0">
@@
 <label x="-741.68" y="266.7" size="1.27" layer="95" xref="yes"/>
 </segment>
-<segment>
-<pinref part="X1" gate="-5" pin="1"/>
-<wire x1="-774.7" y1="160.02" x2="-792.48" y2="160.02" width="0.1524" layer="91"/>
-<label x="-792.48" y="160.02" size="1.27" layer="95" rot="MR0" xref="yes"/>
-</segment>
 </net>
 <net name="STRAND6" class="0">
@@
 <label x="-741.68" y="269.24" size="1.27" layer="95" xref="yes"/>
 </segment>
-<segment>
-<pinref part="X1" gate="-6" pin="1"/>
-<wire x1="-774.7" y1="157.48" x2="-792.48" y2="157.48" width="0.1524" layer="91"/>
-<label x="-792.48" y="157.48" size="1.27" layer="95" rot="MR0" xref="yes"/>
-</segment>
 </net>
 <net name="STRAND7" class="0">
@@
 <label x="-741.68" y="274.32" size="1.27" layer="95" xref="yes"/>
 </segment>
-<segment>
-<pinref part="X1" gate="-7" pin="1"/>
-<wire x1="-774.7" y1="154.94" x2="-792.48" y2="154.94" width="0.1524" layer="91"/>
-<label x="-792.48" y="154.94" size="1.27" layer="95" rot="MR0" xref="yes"/>
-</segment>
 </net>
 <net name="STRAND8" class="0">
@@
 <label x="-741.68" y="281.94" size="1.27" layer="95" xref="yes"/>
 </segment>
-<segment>
-<wire x1="-772.16" y1="152.4" x2="-792.48" y2="152.4" width="0.1524" layer="91"/>
-<label x="-792.48" y="152.4" size="1.27" layer="95" rot="MR0" xref="yes"/>
-</segment>
 </net>
 <net name="STRAND9" class="0">
@@
 <label x="-741.68" y="284.48" size="1.27" layer="95" xref="yes"/>
 </segment>
-<segment>
-<pinref part="X1" gate="-9" pin="1"/>
-<wire x1="-774.7" y1="149.86" x2="-792.48" y2="149.86" width="0.1524" layer="91"/>
-<label x="-792.48" y="149.86" size="1.27" layer="95" rot="MR0" xref="yes"/>
-</segment>
-</net>
+</net>

Commit message: Draft, proofreading required, some components need package changes or value confirmation, board layout and routing required.
Parts:
- added C13, C22: 100n, SmartPrj:C-EUC0603
- added CN1, CN2, CN3, CN4, CN5, CN6: (no value), adafruit:JST_3PIN
- added IC2: LMV358IDGKR, linear:LMV358MMX
- added R13, R14, R15, R16, R17, R18: 300, resistor:R-EU_R0603
- added R19, R20: 10k, SparkFun:RESISTOR0603-RES
- added T1: FDN340P, zetex:PMOSSOT23
- R1: device SmartPrj:R-EU_R0603 -> resistor:R-EU_R0603
Connections:
- removed net AUX_SCL: U4.AUX_CL
- removed net AUX_SDA: U4.AUX_DA
- removed net N$15: U1.(SS/PCINT0)PB0
- removed net STRAND7: U1.(#HWB)PE2
- removed net STRAND8: U1.(OC3A/#0C4A)PC6
- removed net STRAND9: U1.(ICP3/CLK0/OC4A)PC7
- new net CMP: C22.2, IC2B.+IN, R19.1, R20.2
- new net GATE_CMD: IC2B.OUT, T1.G
- new net N$10: CN2.2, R14.2
- new net N$11: CN1.2, R13.2
- new net N$3: CN6.2, R18.2
- new net N$6: CN5.2, R17.2
- new net N$7: CN4.2, R16.2
- new net N$8: CN3.2, R15.2
- net +3V3: now also IC2B.-IN, U2.VREF1
- net +5V: now also C13.1, CN1.1, CN2.1, CN3.1, CN4.1, CN5.1, CN6.1, IC2P.V+, R19.2, T1.S
- net GND: now also C13.2, C22.1, CN1.3, CN2.3, CN3.3, CN4.3, CN5.3, CN6.3, IC2P.V-, R20.1, U1.GND3, U2.GND
- net N$2: now also U2.EN, U2.VREF2
- net SCL1: now also U2.SCL1, U4.SCL; no longer R5.1
- net SCL2: now also U2.SCL2
- net SDA1: now also R5.1, U2.SDA1
- net SDA2: now also U2.SDA2
- net STRAND1: now also R13.1
- net STRAND2: now also R14.1
- net STRAND3: now also R15.1
- net STRAND4: now also R16.1
- net STRAND5: now also R17.1
- net STRAND6: now also R18.1
- net VUSB: now also T1.D
Other:
- note removed: "1. Level shift for MPU logic"
- note removed: "ENABLE tied high, could be IO"
- note removed: "Level-shifter"
- note removed: "LiPo Boost Converter 5v Locked"
- note removed: "Motion Sensor MPU-6050"
- note removed: "Removed 3.3v selector and circuit. Removed output pads. Removed input pads, leaving JST input."
- note removed: "To-Do"
- note removed: "USB"
- note removed: "Why is this?"
- moved on the sheet: C1, C11, C14, C15, C16, C17, C18, C2, C7, C8, C9, J1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
